File: ddr3.kicad_sch (KiCad schematic)
At the start: 6 parts

Commit message: Updating schematics
Other:
- company: (none) -> ${project_creator}
- title: DDR3 -> ${project_name}
Changed lines of the file:
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@@
 	(paper "A3")
 	(title_block
-		(title "DDR3")
-		(date "2024-08-20")
-		(rev "0.0.4")
-		(comment 1 "Reference - ecp5-dc-scm")
+		(title "${project_name}")
+		(date "2025-04-05")
+		(rev "${project_version}")
+		(company "${project_creator}")
+		(comment 1 "${project_license}")
 		(comment 2 "Apache License 2.0")
 	)
