File: ethernet.kicad_sch (KiCad schematic)
At the start: 25 parts, among them U4 LAN8720A

Commit message: Updating schematics
Other:
- company: (none) -> ${project_creator}
- title: Ethernet -> ${project_name}
Changed lines of the file:
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@@
 	(paper "A3")
 	(title_block
-		(title "Ethernet")
-		(date "2024-08-20")
-		(rev "0.0.4")
-		(comment 1 "Reference - ESP32-Ethgate")
+		(title "${project_name}")
+		(date "2025-04-05")
+		(rev "${project_version}")
+		(company "${project_creator}")
+		(comment 1 "${project_license}")
 		(comment 2 "License: CERN-OHL-S v2")
 	)

Commit message: Adding BOM - adding DNP to some components
Parts:
- C85: value 1u1R -> 2.2uF
- R53: value 10K -> 12K1
- R54, R56, R58, R60: value 10R -> 27R
- R55, R57: value 1K5 -> 1K
- R59: value 33R -> 27R
