File: gpdi.kicad_sch (KiCad schematic)
At the start: 45 parts, among them SW1 SW_DIP_x02, U1 LFE5U-85F-6BG381C

Commit message: Updating schematics
Other:
- company: EMARD -> ${project_creator}
- title: ULX3S -> ${project_name}
Changed lines of the file:
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@@
 	(paper "A4")
 	(title_block
-		(title "ULX3S")
-		(date "2024-08-20")
-		(rev "0.0.4")
-		(company "EMARD")
-		(comment 1 "General Purpose Differential Interface")
+		(title "${project_name}")
+		(date "2025-04-05")
+		(rev "${project_version}")
+		(company "${project_creator}")
+		(comment 1 "${project_license}")
 		(comment 2 "License: CERN-OHL-S v2")
 	)

Commit message: Adding BOM - adding DNP to some components
Parts:
- TP_C?, TP_D?: PLACE (none) -> DNP; now not fitted; now left out of the parts list
