File: power.kicad_sch (KiCad schematic)
At the start: 68 parts, among them U1 LFE5U-85F-6BG381C, U5 TLV62569DBV, U6 TLV62569DBV, U7 TLV62569DBV, U8 TLV62569DBV

Commit message: Updating schematics
Other:
- company: EMARD -> ${project_creator}
- title: ULX3S -> ${project_name}
Changed lines of the file:
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@@
 	(paper "A4")
 	(title_block
-		(title "ULX3S")
-		(date "2024-08-20")
-		(rev "0.0.4")
-		(company "EMARD")
-		(comment 1 "Power")
+		(title "${project_name}")
+		(date "2025-04-05")
+		(rev "${project_version}")
+		(company "${project_creator}")
+		(comment 1 "${project_license}")
 		(comment 2 "License: CERN-OHL-S v2")
 	)

Commit message: Adding BOM - adding DNP to some components
Parts:
- 1.1V_1, C? (x6), L4, RA?, RB?, RC?, RP1, RP2, RP3, RP4, RV2, TP_D?, U8: PLACE (none) -> DNP; now not fitted; now left out of the parts list
- C?, D14, R3: PLACE (none) -> DNP
