File: ram.kicad_sch (KiCad schematic)
At the start: 7 parts, among them U1 LFE5U-85F-6BG381C

Commit message: Updating schematics
Other:
- company: Intergalaktik d.o.o. -> ${project_creator}
- title: ULX4M -> ${project_name}
Changed lines of the file:
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@@
 	(paper "A4")
 	(title_block
-		(title "ULX4M")
-		(date "2024-08-20")
-		(rev "0.0.4")
-		(company "Intergalaktik d.o.o.")
-		(comment 1 "SDRAM memory")
+		(title "${project_name}")
+		(date "2025-04-05")
+		(rev "${project_version}")
+		(company "${project_creator}")
+		(comment 1 "${project_license}")
 		(comment 2 "License: CERN-OHL-S v2")
 	)
