File: serdes.kicad_sch (KiCad schematic)
At the start: 26 parts, among them J4 Antenna

Commit message: Updating schematics
Other:
- company: EMARD -> ${project_creator}
- title: ULX3S -> ${project_name}
Changed lines of the file:
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@@
 	(paper "A4")
 	(title_block
-		(title "ULX3S")
-		(date "2024-08-20")
-		(rev "0.0.4")
-		(company "EMARD")
-		(comment 1 "serdes")
+		(title "${project_name}")
+		(date "2025-04-05")
+		(rev "${project_version}")
+		(company "${project_creator}")
+		(comment 1 "${project_license}")
 		(comment 2 "License: CERN-OHL-S v2")
 	)

Commit message: Adding BOM - adding DNP to some components
Parts:
- C? (x4): PLACE (none) -> DNP
- C? (x4), J4: PLACE (none) -> DNP; now not fitted; now left out of the parts list
