File: usb.kicad_sch (KiCad schematic)
At the start: 18 parts, among them J3 JTAG, J6 GPIO>>JTAG, P1 USB_OTG, U1 LFE5U-85F-6BG381C, Y1 FNETHE025

Commit message: Updating schematics
Other:
- company: EMARD -> ${project_creator}
- title: ULX3S -> ${project_name}
Changed lines of the file:
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@@
 	(paper "A4")
 	(title_block
-		(title "ULX3S")
-		(date "2024-08-20")
-		(rev "0.0.4")
-		(company "EMARD")
-		(comment 1 "USB serial and JTAG")
+		(title "${project_name}")
+		(date "2025-04-05")
+		(rev "${project_version}")
+		(company "${project_creator}")
+		(comment 1 "${project_license}")
 		(comment 2 "License: CERN-OHL-S v2")
 	)

Commit message: Adding BOM - adding DNP to some components
Parts:
- J3, J6: PLACE (none) -> DNP; now not fitted; now left out of the parts list
